File: KiCad testing/KiCad testing.kicad_sch (KiCad schematic)
At the start: 35 parts, among them J1 USB_A, Q1 IRF540N, Q2 IRF540N, Q3 IRF540N, U1 IR2113S, U2 IR2113S

Commit message: Update Schematic
Parts:
- U1, U2: footprint Package_SO:SOIC-16W_7.5x10.3mm_P1.27mm -> Package_DIP:DIP-14_W7.62mm_Socket
Connections:
- net GND: no longer J1.4 (GND)
Other:
- moved on the sheet: C1, C5, D1, L2, Q1

Commit message: Update Schematic
Parts:
- added R10, R12: 1k, symbol Device:R_US
- added R11, R9: 1400, symbol Device:R_US
- added SC1: Solar_Cells, symbol Device:Solar_Cells
- added U3: ACS712xLCTR-05B, Package_SO:SOIC-8_3.9x4.9mm_P1.27mm, symbol Sensor_Current:ACS712xLCTR-05B
Connections:
- net 5V: now also U3.8 (VCC)
- net GND: now also R10.2, R12.2, U3.5 (GND)
- net Battery_Voltage: now reaches A1.19 (A0)
- net Battery_Voltage: now also R11.2, R12.1
- net Battery_V_Sensor: now reaches BT1.1 (+), C12.1, L1.2
- net Battery_V_Sensor: now also R11.1
- new net: U3.1 (IP+), U3.2 (IP+)
- new net: U3.3 (IP-), U3.4 (IP-)
- new net PV_V_Sensor: R9.1
- new net PV_Voltage: R10.1, R9.2

Commit message: Update Schematic
Parts:
- C1, C2, C5: footprint (none) -> Capacitor_THT:CP_Radial_D6.3mm_P2.50mm
- C12: footprint (none) -> Capacitor_THT:CP_Radial_D10.0mm_P5.00mm
- L1, L2: footprint (none) -> Inductor_THT:L_Radial_D10.5mm_P5.00mm_Abacron_AISR-01
- R1, R10, R12, R2, R3, R4, R5, R6, R7, R8: footprint (none) -> Resistor_THT:R_Axial_DIN0207_L6.3mm_D2.5mm_P10.16mm_Horizontal
Connections:
- net PV_Voltage: now also A1.20 (A1)
- net PV_Current: now reaches A1.21 (A2)
- net at U3.1 (IP+), U3.2 (IP+): now also SC1.1 (+)
- net at U3.3 (IP-), U3.4 (IP-): now also SC1.2 (-)
Changed lines of the file:
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@@
+    (stroke (width 0) (type default))
+  )
+  (wire (pts (xy 78.74 163.83) (xy 100.33 163.83))
     (stroke (width 0) (type default))
   )
@@
   )
   (wire (pts (xy 207.01 48.26) (xy 220.98 48.26))
+    (stroke (width 0) (type default))
+  )
+  (wire (pts (xy 78.74 153.67) (xy 100.33 153.67))
     (stroke (width 0) (type default))
   )
@@
     )
   )
+  (global_label "PV_Current" (shape input) (at 50.8 49.53 0) (fields_autoplaced)
+    (effects (font (size 1.27 1.27)) (justify left))
+    (property "Intersheetrefs" "${INTERSHEET_REFS}" (at 63.4119 49.53 0)
+      (effects (font (size 1.27 1.27)) (justify left) hide)
+    )
+  )
   (global_label "GND" (shape input) (at 20.32 186.69 270)
     (effects (font (size 1.27 1.27)) (justify right))
@@
     (property "Intersheetrefs" "${INTERSHEET_REFS}" (at 73.66 99.06 0)
       (effects (font (size 1.27 1.27)) hide)
+    )
+  )
+  (global_label "PV_Voltage" (shape input) (at 50.8 46.99 0) (fields_autoplaced)
+    (effects (font (size 1.27 1.27)) (justify left))
+    (property "Intersheetrefs" "${INTERSHEET_REFS}" (at 63.4723 46.99 0)
+      (effects (font (size 1.27 1.27)) (justify left) hide)
     )
   )
@@
       (effects (font (size 1.27 1.27)))
     )
-    (property "Footprint" "" (at 98.044 33.274 90)
+    (property "Footprint" "Resistor_THT:R_Axial_DIN0207_L6.3mm_D2.5mm_P10.16mm_Horizontal" (at 98.044 33.274 90)
       (effects (font (size 1.27 1.27)) hide)
     )
@@
       (effects (font (size 1.27 1.27)))
     )
-    (property "Footprint" "" (at 103.124 59.436 90)
+    (property "Footprint" "Resistor_THT:R_Axial_DIN0207_L6.3mm_D2.5mm_P10.16mm_Horizontal" (at 103.124 59.436 90)
       (effects (font (size 1.27 1.27)) hide)
     )
@@
       (effects (font (size 1.27 1.27)))
     )
-    (property "Footprint" "" (at 101.854 37.846 90)
+    (property "Footprint" "Resistor_THT:R_Axial_DIN0207_L6.3mm_D2.5mm_P10.16mm_Horizontal" (at 101.854 37.846 90)
       (effects (font (size 1.27 1.27)) hide)
     )
@@
       (effects (font (size 1.27 1.27)))
     )
-    (property "Footprint" "" (at 96.266 55.626 90)
+    (property "Footprint" "Resistor_THT:R_Axial_DIN0207_L6.3mm_D2.5mm_P10.16mm_Horizontal" (at 96.266 55.626 90)
       (effects (font (size 1.27 1.27)) hide)
     )
@@
       (effects (font (size 1.27 1.27)))
     )
-    (property "Footprint" "" (at 98.044 87.884 90)
+    (property "Footprint" "Resistor_THT:R_Axial_DIN0207_L6.3mm_D2.5mm_P10.16mm_Horizontal" (at 98.044 87.884 90)
       (effects (font (size 1.27 1.27)) hide)
     )
@@
       (effects (font (size 1.27 1.27)))
     )
-    (property "Footprint" "" (at 103.124 114.046 90)
+    (property "Footprint" "Resistor_THT:R_Axial_DIN0207_L6.3mm_D2.5mm_P10.16mm_Horizontal" (at 103.124 114.046 90)
       (effects (font (size 1.27 1.27)) hide)
     )
@@
       (effects (font (size 1.27 1.27)))
     )
-    (property "Footprint" "" (at 101.854 92.456 90)
+    (property "Footprint" "Resistor_THT:R_Axial_DIN0207_L6.3mm_D2.5mm_P10.16mm_Horizontal" (at 101.854 92.456 90)
       (effects (font (size 1.27 1.27)) hide)
     )
@@
       (effects (font (size 1.27 1.27)))
     )
-    (property "Footprint" "" (at 96.266 110.236 90)
+    (property "Footprint" "Resistor_THT:R_Axial_DIN0207_L6.3mm_D2.5mm_P10.16mm_Horizontal" (at 96.266 110.236 90)
       (effects (font (size 1.27 1.27)) hide)
     )
@@
       (effects (font (size 1.27 1.27)) (justify left))
     )
-    (property "Footprint" "" (at 175.26 44.45 0)
+    (property "Footprint" "Capacitor_THT:CP_Radial_D6.3mm_P2.50mm" (at 175.26 44.45 0)
       (effects (font (size 1.27 1.27)) hide)
     )
@@
       (effects (font (size 1.27 1.27)) (justify left))
     )
-    (property "Footprint" "" (at 233.68 44.45 0)
+    (property "Footprint" "Capacitor_THT:CP_Radial_D10.0mm_P5.00mm" (at 233.68 44.45 0)
       (effects (font (size 1.27 1.27)) hide)
     )
@@
       (effects (font (size 1.27 1.27)))
     )
-    (property "Footprint" "" (at 227.33 38.1 0)
+    (property "Footprint" "Inductor_THT:L_Radial_D10.5mm_P5.00mm_Abacron_AISR-01" (at 227.33 38.1 0)
       (effects (font (size 1.27 1.27)) hide)
     )
@@
       (effects (font (size 1.27 1.27)))
     )
-    (property "Footprint" "" (at 46.736 183.134 90)
+    (property "Footprint" "Resistor_THT:R_Axial_DIN0207_L6.3mm_D2.5mm_P10.16mm_Horizontal" (at 46.736 183.134 90)
       (effects (font (size 1.27 1.27)) hide)
     )
@@
       (effects (font (size 1.27 1.27)) (justify left))
     )
-    (property "Footprint" "" (at 170.18 80.01 0)
+    (property "Footprint" "Capacitor_THT:CP_Radial_D6.3mm_P2.50mm" (at 170.18 80.01 0)
       (effects (font (size 1.27 1.27)) hide)
     )
@@
       (effects (font (size 1.27 1.27)) (justify left))
     )
-    (property "Footprint" "" (at 213.36 80.01 0)
+    (property "Footprint" "Capacitor_THT:CP_Radial_D6.3mm_P2.50mm" (at 213.36 80.01 0)
       (effects (font (size 1.27 1.27)) hide)
     )
@@
       (effects (font (size 1.27 1.27)))
     )
-    (property "Footprint" "" (at 21.336 183.134 90)
+    (property "Footprint" "Resistor_THT:R_Axial_DIN0207_L6.3mm_D2.5mm_P10.16mm_Horizontal" (at 21.336 183.134 90)
       (effects (font (size 1.27 1.27)) hide)
     )
@@
       (effects (font (size 1.27 1.27)))
     )
-    (property "Footprint" "" (at 199.39 80.01 0)
-      (effects (font (size 1.27 1.27)) hide)
-    )
+    (property "Footprint" "Inductor_THT:L_Radial_D10.5mm_P5.00mm_Abacron_AISR-01" (at 199.39 80.01 0)
+      (effects (font (size 1.27 1.27)) hide)
+    )
