File: KiCad testing/_autosave-KiCad testing.kicad_sch (KiCad schematic)
At the start: 41 parts, among them J1 USB_A, Q1 IRF540N, Q2 IRF540N, Q3 IRF540N, U1 IR2113S, U2 IR2113S, U3 ACS712xLCTR-05B

Commit message: Update Schematic
Begin PCB layout. Not final design.
Parts:
- renumbered C6 to C1, C12 to C10, C1 to C11, C5 to C12, C9 to C2, C7 to C5, C10 to C6, C11 to C7, C2 to C9, D2 to D1, D3 to D2, D5 to D3, D1 to D5, R5 to R2, R2 to R4, R6 to R5, R4 to R6, R9 to Rb1, R11 to Rb2
Connections:
- net VS: no longer C6.2, R5.1, U2.6 (VS)
- new net VS_1: C6.2, R5.1, U2.6 (VS)
Changed lines of the file:
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@@
     )
   )
-  (global_label "VS" (shape output) (at 106.68 100.33 270)
+  (global_label "VS_1" (shape output) (at 106.68 100.33 270)
     (effects (font (size 1.27 1.27)) (justify right))
     (property "Intersheetrefs" "${INTERSHEET_REFS}" (at 106.68 100.33 0)
@@
   (symbol (lib_id "Diode:1N4148") (at 120.65 36.83 0) (unit 1)
     (in_bom yes) (on_board yes) (dnp no)
-    (property "Reference" "D2" (at 120.65 42.3164 0)
+    (property "Reference" "D1" (at 120.65 42.3164 0)
       (effects (font (size 1.27 1.27)))
     )
@@
       (project "KiCad testing"
         (path "/7cafa5f9-ca51-4b5e-ba3d-0c99ad1b0c30"
-          (reference "D2") (unit 1)
+          (reference "D1") (unit 1)
         )
       )
@@
   (symbol (lib_id "KiCad testing-rescue:CP1-Device") (at 85.09 58.42 180) (unit 1)
     (in_bom yes) (on_board yes) (dnp no)
-    (property "Reference" "C6" (at 88.011 57.2516 0)
+    (property "Reference" "C1" (at 88.011 57.2516 0)
       (effects (font (size 1.27 1.27)) (justify right))
     )
@@
       (project "KiCad testing"
         (path "/7cafa5f9-ca51-4b5e-ba3d-0c99ad1b0c30"
-          (reference "C6") (unit 1)
+          (reference "C1") (unit 1)
         )
       )
@@
   (symbol (lib_id "Device:R_US") (at 106.68 38.1 180) (unit 1)
     (in_bom yes) (on_board yes) (dnp no)
-    (property "Reference" "R5" (at 101.473 38.1 90)
+    (property "Reference" "R2" (at 101.473 38.1 90)
       (effects (font (size 1.27 1.27)))
     )
@@
       (project "KiCad testing"
         (path "/7cafa5f9-ca51-4b5e-ba3d-0c99ad1b0c30"
-          (reference "R5") (unit 1)
+          (reference "R2") (unit 1)
         )
       )
@@
   (symbol (lib_id "Device:R_US") (at 101.6 88.9 90) (unit 1)
     (in_bom yes) (on_board yes) (dnp no)
-    (property "Reference" "R4" (at 101.6 83.693 90)
+    (property "Reference" "R6" (at 101.6 83.693 90)
       (effects (font (size 1.27 1.27)))
     )
@@
       (project "KiCad testing"
         (path "/7cafa5f9-ca51-4b5e-ba3d-0c99ad1b0c30"
-          (reference "R4") (unit 1)
+          (reference "R6") (unit 1)
         )
       )
@@
   (symbol (lib_id "KiCad testing-rescue:CP1-Device") (at 85.09 113.03 180) (unit 1)
     (in_bom yes) (on_board yes) (dnp no)
-    (property "Reference" "C7" (at 88.011 111.8616 0)
+    (property "Reference" "C5" (at 88.011 111.8616 0)
       (effects (font (size 1.27 1.27)) (justify right))
     )
@@
       (project "KiCad testing"
         (path "/7cafa5f9-ca51-4b5e-ba3d-0c99ad1b0c30"
-          (reference "C7") (unit 1)
+          (reference "C5") (unit 1)
         )
       )
@@
   (symbol (lib_id "Device:R_US") (at 106.68 92.71 180) (unit 1)
     (in_bom yes) (on_board yes) (dnp no)
-    (property "Reference" "R6" (at 101.473 92.71 90)
+    (property "Reference" "R5" (at 101.473 92.71 90)
       (effects (font (size 1.27 1.27)))
     )
@@
       (project "KiCad testing"
         (path "/7cafa5f9-ca51-4b5e-ba3d-0c99ad1b0c30"
-          (reference "R6") (unit 1)
+          (reference "R5") (unit 1)
         )
       )
@@
   (symbol (lib_id "Device:R_US") (at 100.33 109.22 270) (unit 1)
     (in_bom yes) (on_board yes) (dnp no)
-    (property "Reference" "R2" (at 100.33 114.427 90)
+    (property "Reference" "R4" (at 100.33 114.427 90)
       (effects (font (size 1.27 1.27)))
     )
@@
       (project "KiCad testing"
         (path "/7cafa5f9-ca51-4b5e-ba3d-0c99ad1b0c30"
-          (reference "R2") (unit 1)
+          (reference "R4") (unit 1)
         )
       )
@@
   (symbol (lib_id "KiCad testing-rescue:CP1-Device") (at 123.19 82.55 180) (unit 1)
     (in_bom yes) (on_board yes) (dnp no)
-    (property "Reference" "C11" (at 126.111 81.3816 0)
+    (property "Reference" "C7" (at 126.111 81.3816 0)
       (effects (font (size 1.27 1.27)) (justify right))
     )
@@
       (project "KiCad testing"
         (path "/7cafa5f9-ca51-4b5e-ba3d-0c99ad1b0c30"
-          (reference "C11") (unit 1)
+          (reference "C7") (unit 1)
         )
       )
@@
   (symbol (lib_id "KiCad testing-rescue:CP1-Device") (at 113.03 96.52 270) (unit 1)
     (in_bom yes) (on_board yes) (dnp no)
-    (property "Reference" "C10" (at 111.8616 93.599 0)
+    (property "Reference" "C6" (at 111.8616 93.599 0)
       (effects (font (size 1.27 1.27)) (justify right))
     )
@@
       (project "KiCad testing"
         (path "/7cafa5f9-ca51-4b5e-ba3d-0c99ad1b0c30"
-          (reference "C10") (unit 1)
+          (reference "C6") (unit 1)
         )
       )
@@
   (symbol (lib_id "Diode:1N4148") (at 120.65 91.44 0) (unit 1)
     (in_bom yes) (on_board yes) (dnp no)
-    (property "Reference" "D3" (at 120.65 96.9264 0)
+    (property "Reference" "D2" (at 120.65 96.9264 0)
       (effects (font (size 1.27 1.27)))
     )
@@
       (project "KiCad testing"
         (path "/7cafa5f9-ca51-4b5e-ba3d-0c99ad1b0c30"
-          (reference "D3") (unit 1)
+          (reference "D2") (unit 1)
         )
       )
@@
   (symbol (lib_id "KiCad testing-rescue:CP1-Device") (at 175.26 44.45 0) (unit 1)
     (in_bom yes) (on_board yes) (dnp no)
-    (property "Reference" "C2" (at 178.181 43.2816 0)
+    (property "Reference" "C9" (at 178.181 43.2816 0)
       (effects (font (size 1.27 1.27)) (justify left))
     )
@@
       (project "KiCad testing"
         (path "/7cafa5f9-ca51-4b5e-ba3d-0c99ad1b0c30"
-          (reference "C2") (unit 1)
+          (reference "C9") (unit 1)
         )
       )
@@
   (symbol (lib_id "Diode:1N4002") (at 220.98 44.45 270) (unit 1)
     (in_bom yes) (on_board yes) (dnp no)
-    (property "Reference" "D5" (at 226.4664 44.45 0)
+    (property "Reference" "D3" (at 226.4664 44.45 0)
       (effects (font (size 1.27 1.27)))
     )
@@
       (project "KiCad testing"
         (path "/7cafa5f9-ca51-4b5e-ba3d-0c99ad1b0c30"
-          (reference "D5") (unit 1)
+          (reference "D3") (unit 1)
         )
       )
@@
   (symbol (lib_id "KiCad testing-rescue:CP1-Device") (at 233.68 44.45 0) (unit 1)
     (in_bom yes) (on_board yes) (dnp no)
-    (property "Reference" "C12" (at 236.601 43.2816 0)
+    (property "Reference" "C10" (at 236.601 43.2816 0)
       (effects (font (size 1.27 1.27)) (justify left))
     )
@@
       (project "KiCad testing"
         (path "/7cafa5f9-ca51-4b5e-ba3d-0c99ad1b0c30"
-          (reference "C12") (unit 1)
+          (reference "C10") (unit 1)
         )
       )
@@
   (symbol (lib_id "KiCad testing-rescue:CP1-Device") (at 170.18 80.01 0) (unit 1)
     (in_bom yes) (on_board yes) (dnp no)
-    (property "Reference" "C5" (at 173.101 78.8416 0)
+    (property "Reference" "C12" (at 173.101 78.8416 0)
       (effects (font (size 1.27 1.27)) (justify left))
     )
@@
       (project "KiCad testing"
         (path "/7cafa5f9-ca51-4b5e-ba3d-0c99ad1b0c30"
-          (reference "C5") (unit 1)
+          (reference "C12") (unit 1)
         )
       )
@@
   (symbol (lib_id "KiCad testing-rescue:CP1-Device") (at 213.36 80.01 180) (unit 1)
     (in_bom yes) (on_board yes) (dnp no)
-    (property "Reference" "C1" (at 210.439 81.1784 0)
+    (property "Reference" "C11" (at 210.439 81.1784 0)
       (effects (font (size 1.27 1.27)) (justify left))
     )
@@
       (project "KiCad testing"
         (path "/7cafa5f9-ca51-4b5e-ba3d-0c99ad1b0c30"
-          (reference "C1") (unit 1)
+          (reference "C11") (unit 1)
         )
       )
@@
   (symbol (lib_id "Diode:1N4002") (at 207.01 73.66 0) (unit 1)
     (in_bom yes) (on_board yes) (dnp no)
-    (property "Reference" "D1" (at 207.01 68.1736 0)
+    (property "Reference" "D5" (at 207.01 68.1736 0)
       (effects (font (size 1.27 1.27)))
     )
@@
       (project "KiCad testing"
         (path "/7cafa5f9-ca51-4b5e-ba3d-0c99ad1b0c30"
-          (reference "D1") (unit 1)
+          (reference "D5") (unit 1)
         )
       )
@@
   (symbol (lib_id "Device:R_US") (at 29.21 99.06 0) (unit 1)
     (in_bom yes) (on_board yes) (dnp no)
-    (property "Reference" "R9" (at 34.417 99.06 90)
+    (property "Reference" "Rb1" (at 34.417 99.06 90)
       (effects (font (size 1.27 1.27)))
     )
@@
       (project "KiCad testing"
         (path "/7cafa5f9-ca51-4b5e-ba3d-0c99ad1b0c30"
-          (reference "R9") (unit 1)
+          (reference "Rb1") (unit 1)
         )
       )
@@
   (symbol (lib_id "Device:R_US") (at 45.72 99.06 0) (unit 1)
     (in_bom yes) (on_board yes) (dnp no)
-    (property "Reference" "R11" (at 50.927 99.06 90)
+    (property "Reference" "Rb2" (at 50.927 99.06 90)
       (effects (font (size 1.27 1.27)))
     )
@@
       (project "KiCad testing"
         (path "/7cafa5f9-ca51-4b5e-ba3d-0c99ad1b0c30"
-          (reference "R11") (unit 1)
+          (reference "Rb2") (unit 1)
         )
       )
@@
   (symbol (lib_id "KiCad testing-rescue:CP1-Device") (at 113.03 41.91 270) (unit 1)
     (in_bom yes) (on_board yes) (dnp no)
-    (property "Reference" "C9" (at 111.8616 38.989 0)
+    (property "Reference" "C2" (at 111.8616 38.989 0)
       (effects (font (size 1.27 1.27)) (justify right))
     )
@@
       (project "KiCad testing"
         (path "/7cafa5f9-ca51-4b5e-ba3d-0c99ad1b0c30"
-          (reference "C9") (unit 1)
-        )
-      )
+          (reference "C2") (unit 1)
+        )
+      )
